File: nanofloat-pressure-sensor-mount/nanofloat-pressure-sensor-mount.kicad_sch (KiCad schematic)
At the start: 2 parts, among them J1 Conn_01x04_Pin

Commit message: Updating KiCAD project files
Parts:
- J1: footprint Connector_PinHeader_1.00mm:PinHeader_1x04_P1.00mm_Vertical -> Connector_PinHeader_2.54mm:PinHeader_1x04_P2.54mm_Vertical
Connections:
- new net: J1.1 (Pin_1), U1.1 (GND)
- new net: J1.2 (Pin_2), U1.2 (VDD)
- new net: J1.3 (Pin_3), U1.3 (SCL)
- new net: J1.4 (Pin_4), U1.4 (SDA)
Changed lines of the file:
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@@
 (kicad_sch (version 20230121) (generator eeschema)
   (paper "A4")
-  (junction (at 160.02 92.71) (diameter 0) (color 0 0 0 0)
-  )
-  (junction (at 140.97 90.17) (diameter 0) (color 0 0 0 0)
-  )
-  (junction (at 140.97 87.63) (diameter 0) (color 0 0 0 0)
-  )
-  (junction (at 119.38 107.95) (diameter 0) (color 0 0 0 0)
-  )
-  (junction (at 140.97 92.71) (diameter 0) (color 0 0 0 0)
-  )
-  (junction (at 160.02 107.95) (diameter 0) (color 0 0 0 0)
-  )
-  (wire (pts (xy 140.97 90.17) (xy 160.02 90.17))
-    (stroke (width 0) (type default))
-  )
-  (wire (pts (xy 140.97 107.95) (xy 119.38 107.95))
-    (stroke (width 0) (type default))
-  )
-  (wire (pts (xy 140.97 90.17) (xy 140.97 92.71))
-    (stroke (width 0) (type default))
-  )
-  (wire (pts (xy 160.02 92.71) (xy 160.02 107.95))
-    (stroke (width 0) (type default))
-  )
-  (wire (pts (xy 140.97 85.09) (xy 140.97 87.63))
-    (stroke (width 0) (type default))
-  )
-  (wire (pts (xy 160.02 107.95) (xy 160.02 110.49))
-    (stroke (width 0) (type default))
-  )
   (wire (pts (xy 140.97 92.71) (xy 160.02 92.71))
     (stroke (width 0) (type default))
   )
-  (wire (pts (xy 140.97 87.63) (xy 140.97 90.17))
+  (wire (pts (xy 162.56 110.49) (xy 160.02 110.49))
     (stroke (width 0) (type default))
   )
-  (wire (pts (xy 119.38 87.63) (xy 119.38 107.95))
+  (wire (pts (xy 147.32 76.2) (xy 147.32 87.63))
     (stroke (width 0) (type default))
   )
-  (wire (pts (xy 140.97 92.71) (xy 140.97 107.95))
+  (wire (pts (xy 147.32 87.63) (xy 140.97 87.63))
     (stroke (width 0) (type default))
   )
-  (wire (pts (xy 160.02 90.17) (xy 160.02 92.71))
+  (wire (pts (xy 160.02 107.95) (xy 160.02 92.71))
     (stroke (width 0) (type default))
   )
-  (wire (pts (xy 140.97 87.63) (xy 119.38 87.63))
+  (wire (pts (xy 140.97 90.17) (xy 162.56 90.17))
     (stroke (width 0) (type default))
   )
-  (wire (pts (xy 119.38 107.95) (xy 119.38 110.49))
+  (wire (pts (xy 162.56 90.17) (xy 162.56 110.49))
+    (stroke (width 0) (type default))
+  )
+  (wire (pts (xy 119.38 107.95) (xy 119.38 77.47))
+    (stroke (width 0) (type default))
+  )
+  (wire (pts (xy 146.05 77.47) (xy 146.05 85.09))
+    (stroke (width 0) (type default))
+  )
+  (wire (pts (xy 119.38 110.49) (xy 118.11 110.49))
+    (stroke (width 0) (type default))
+  )
+  (wire (pts (xy 118.11 76.2) (xy 147.32 76.2))
+    (stroke (width 0) (type default))
+  )
+  (wire (pts (xy 119.38 77.47) (xy 146.05 77.47))
+    (stroke (width 0) (type default))
+  )
+  (wire (pts (xy 118.11 110.49) (xy 118.11 76.2))
+    (stroke (width 0) (type default))
+  )
+  (wire (pts (xy 146.05 85.09) (xy 140.97 85.09))
     (stroke (width 0) (type default))
   )
@@
       (effects (font (size 1.27 1.27)))
     )
-    (property "Footprint" "Connector_PinHeader_1.00mm:PinHeader_1x04_P1.00mm_Vertical" (at 135.89 87.63 0)
+    (property "Footprint" "Connector_PinHeader_2.54mm:PinHeader_1x04_P2.54mm_Vertical" (at 135.89 87.63 0)
       (effects (font (size 1.27 1.27)) hide)
     )
