File: Pressure_Sensor_Mount/v0.2/Pressure_Sensor_Mount_v0.2.kicad_pcb (KiCad board)
At the start: 2 copper layers, 18.4 x 13.6 mm, 5 parts, among them J1 Conn_01x04_Pin

Commit message: Updated PSM v0.2
Parts:
- moved C1 0.75 mm to (141.1, 86.5)
- moved J1 0.40 mm to (155.6, 87.3)
Routing:
- net Net-(J1-Pin_3): track 19.9 -> 15.7 mm
- net Net-(J1-Pin_2): track 42.2 -> 40.9 mm
- net Net-(J1-Pin_1): track 16.5 -> 15.5 mm
Other:
- board size 18.4 x 13.6 mm -> 18.4 x 12.8 mm
Changed lines of the file:
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@@
   (net 4 "Net-(J1-Pin_4)")
   (footprint "Capacitor_THT:C_Disc_D3.0mm_W1.6mm_P2.50mm" (layer "F.Cu")
-    (at 141.1 85.75 -90)
+    (at 141.1 86.5 -90)
     (descr "C, Disc series, Radial, pin pitch=2.50mm, , diameter*width=3.0*1.6mm^2, Capacitor, http://www.vishay.com/docs/45233/krseries.pdf")
     (tags "C Disc series Radial pin pitch 2.50mm  diameter 3.0mm width 1.6mm Capacitor")
@@
     (property "ki_keywords" "capacitor cap")
     (attr through_hole)
-    (fp_text reference "C1" (at 4.15 0.4 -180) (layer "F.SilkS")
+    (fp_text reference "C1" (at 4.1 0.5 -180) (layer "F.SilkS")
         (effects (font (size 0.8 0.8) (thickness 0.1)))
     )
@@
     (property "ki_keywords" "MS583730BA01-50")
     (attr smd)
-    (fp_text reference "U1" (at 0.000001 -2.699999 unlocked) (layer "F.SilkS") hide
-        (effects (font (size 1 1) (thickness 0.15)))
+    (fp_text reference "U1" (at 0.100001 0.000001 unlocked) (layer "F.SilkS") hide
+        (effects (font (size 0.8 0.8) (thickness 0.1)))
     )
     (fp_text value "~" (at 0.00325 -0.000001 unlocked) (layer "F.Fab") hide
@@
     (fp_line (start 1.8796 1.8796) (end 1.8796 -1.8796)
       (stroke (width 0.1524) (type solid)) (layer "F.SilkS"))
-    (fp_circle (center -2.5969 -1) (end -2.5207 -1)
-      (stroke (width 0.1524) (type solid)) (fill none) (layer "F.SilkS"))
     (fp_poly
       (pts
@@
   )
   (footprint "Connector_PinHeader_2.54mm:PinHeader_1x04_P2.54mm_Vertical" (layer "B.Cu")
-    (at 155.62 86.9 90)
+    (at 155.62 87.3 90)
     (descr "Through hole straight pin header, 1x04, 2.54mm pitch, single row")
     (tags "Through hole pin header THT 1x04 2.54mm single row")
@@
     )
   )
-  (gr_rect (start 139.5 84.2) (end 157.9 97.8)
+  (gr_rect (start 139.5 85) (end 157.9 97.8)
     (stroke (width 0.1) (type default)) (fill none) (layer "Edge.Cuts"))
-  (gr_text "GND" (at 157 89.4) (layer "B.SilkS")
+  (gr_text "GND" (at 157 89.8) (layer "B.SilkS")
     (effects (font (size 0.8 0.8) (thickness 0.1)) (justify left bottom mirror))
   )
-  (gr_text "SDA" (at 149.3 89.4) (layer "B.SilkS")
+  (gr_text "SDA" (at 149.3 89.8) (layer "B.SilkS")
     (effects (font (size 0.8 0.8) (thickness 0.1)) (justify left bottom mirror))
   )
-  (gr_text "SCL" (at 151.8 89.4) (layer "B.SilkS")
+  (gr_text "SCL" (at 151.8 89.8) (layer "B.SilkS")
     (effects (font (size 0.8 0.8) (thickness 0.1)) (justify left bottom mirror))
   )
-  (gr_text "VDD" (at 154.3 89.4) (layer "B.SilkS")
+  (gr_text "VDD" (at 154.3 89.8) (layer "B.SilkS")
     (effects (font (size 0.8 0.8) (thickness 0.1)) (justify left bottom mirror))
   )
@@
     (effects (font (size 0.8 0.8) (thickness 0.1)) (justify left bottom))
   )
-  (gr_text "VDD" (at 151.9 85.4) (layer "F.SilkS")
-    (effects (font (size 0.8 0.8) (thickness 0.1)) (justify left bottom))
-  )
-  (gr_text "SDA" (at 146.8 85.4) (layer "F.SilkS")
-    (effects (font (size 0.8 0.8) (thickness 0.1)) (justify left bottom))
-  )
-  (gr_text "GND" (at 154.4 85.4) (layer "F.SilkS")
-    (effects (font (size 0.8 0.8) (thickness 0.1)) (justify left bottom))
-  )
-  (gr_text "SCL" (at 149.4 85.4) (layer "F.SilkS")
-    (effects (font (size 0.8 0.8) (thickness 0.1)) (justify left bottom))
-  )
-  (segment (start 144.274996 85.725) (end 144.275 85.725) (width 0.25) (layer "F.Cu") (net 1))
-  (segment (start 145 85) (end 153.72 85) (width 0.25) (layer "F.Cu") (net 1))
-  (segment (start 153.72 85) (end 155.62 86.9) (width 0.25) (layer "F.Cu") (net 1))
-  (segment (start 142.149998 86.799998) (end 141.1 85.75) (width 0.25) (layer "F.Cu") (net 1))
-  (segment (start 144.275 85.725) (end 145 85) (width 0.25) (layer "F.Cu") (net 1))
-  (segment (start 143.199998 86.799998) (end 142.149998 86.799998) (width 0.25) (layer "F.Cu") (net 1))
-  (segment (start 143.199998 86.799998) (end 144.274996 85.725) (width 0.25) (layer "F.Cu") (net 1))
-  (segment (start 153.08 86.9) (end 156.2 90.02) (width 0.25) (layer "F.Cu") (net 2))
-  (segment (start 141.1 88.25) (end 141.1 93.1) (width 0.25) (layer "F.Cu") (net 2))
+  (gr_text "VDD" (at 152 89.8) (layer "F.SilkS")
+    (effects (font (size 0.8 0.8) (thickness 0.1)) (justify left bottom))
+  )
+  (gr_text "SDA" (at 146.9 89.8) (layer "F.SilkS")
+    (effects (font (size 0.8 0.8) (thickness 0.1)) (justify left bottom))
+  )
+  (gr_text "GND" (at 154.5 89.8) (layer "F.SilkS")
+    (effects (font (size 0.8 0.8) (thickness 0.1)) (justify left bottom))
+  )
+  (gr_text "SCL" (at 149.5 89.8) (layer "F.SilkS")
+    (effects (font (size 0.8 0.8) (thickness 0.1)) (justify left bottom))
+  )
+  (segment (start 142.9 86.5) (end 143.199998 86.799998) (width 0.25) (layer "F.Cu") (net 1))
+  (segment (start 143.199998 86.799998) (end 144.020298 85.979698) (width 0.25) (layer "F.Cu") (net 1))
+  (segment (start 144.020298 85.979698) (end 154.299698 85.979698) (width 0.25) (layer "F.Cu") (net 1))
+  (segment (start 154.299698 85.979698) (end 155.62 87.3) (width 0.25) (layer "F.Cu") (net 1))
+  (segment (start 141.1 86.5) (end 142.9 86.5) (width 0.25) (layer "F.Cu") (net 1))
   (segment (start 142.375 89.624998) (end 142.375 92.175) (width 0.25) (layer "F.Cu") (net 2))
   (segment (start 141.1 93.1) (end 143.5 95.5) (width 0.25) (layer "F.Cu") (net 2))
-  (segment (start 156.2 90.02) (end 156.2 91.7) (width 0.25) (layer "F.Cu") (net 2))
+  (segment (start 153.08 88.58) (end 156.2 91.7) (width 0.25) (layer "F.Cu") (net 2))
   (segment (start 146.825 96.625) (end 156.75 96.625) (width 0.25) (layer "F.Cu") (net 2))
   (segment (start 157.325 96.05) (end 157.325 92.825) (width 0.25) (layer "F.Cu") (net 2))
   (segment (start 143.199998 88.8) (end 142.375 89.624998) (width 0.25) (layer "F.Cu") (net 2))
   (segment (start 142.375 92.175) (end 146.825 96.625) (width 0.25) (layer "F.Cu") (net 2))
+  (segment (start 142.999998 89) (end 143.199998 88.8) (width 0.25) (layer "F.Cu") (net 2))
+  (segment (start 153.08 87.3) (end 153.08 88.58) (width 0.25) (layer "F.Cu") (net 2))
+  (segment (start 141.1 89) (end 142.999998 89) (width 0.25) (layer "F.Cu") (net 2))
   (segment (start 157.325 92.825) (end 156.2 91.7) (width 0.25) (layer "F.Cu") (net 2))
-  (segment (start 143.199998 88.8) (end 141.65 88.8) (width 0.25) (layer "F.Cu") (net 2))
+  (segment (start 141.1 89) (end 141.1 93.1) (width 0.25) (layer "F.Cu") (net 2))
   (segment (start 156.75 96.625) (end 157.325 96.05) (width 0.25) (layer "F.Cu") (net 2))
-  (segment (start 141.65 88.8) (end 141.1 88.25) (width 0.25) (layer "F.Cu") (net 2))
   (segment (start 149.5 88.8) (end 156.2 95.5) (width 0.25) (layer "F.Cu") (net 3))
-  (segment (start 148.64 88.8) (end 150.54 86.9) (width 0.25) (layer "F.Cu") (net 3))
   (segment (start 145.2 88.8) (end 149.5 88.8) (width 0.25) (layer "F.Cu") (net 3))
-  (segment (start 145.2 88.8) (end 148.64 88.8) (width 0.25) (layer "F.Cu") (net 3))
+  (segment (start 150.54 87.3) (end 149.5 88.34) (width 0.25) (layer "F.Cu") (net 3))
+  (segment (start 149.5 88.34) (end 149.5 88.8) (width 0.25) (layer "F.Cu") (net 3))
   (segment (start 145.2 86.799998) (end 144.3797 87.620298) (width 0.25) (layer "F.Cu") (net 4))
   (segment (start 144.3797 90.8203) (end 143.5 91.7) (width 0.25) (layer "F.Cu") (net 4))
-  (segment (start 145.2 86.799998) (end 147.899998 86.799998) (width 0.25) (layer "F.Cu") (net 4))
+  (segment (start 145.700002 87.3) (end 145.2 86.799998) (width 0.25) (layer "F.Cu") (net 4))
+  (segment (start 148 87.3) (end 145.700002 87.3) (width 0.25) (layer "F.Cu") (net 4))
   (segment (start 147.899998 86.799998) (end 148 86.9) (width 0.25) (layer "F.Cu") (net 4))
   (segment (start 144.3797 87.620298) (end 144.3797 90.8203) (width 0.25) (layer "F.Cu") (net 4))
