File: Nano-Float_Schematic/Nano-Float_Schematic.kicad_pcb (KiCad board)
At the start: 2 copper layers, 25.6 x 53.3 mm, 8 parts, among them M1 Motor_DC, SW1 SW_DIP_x01, U1 MS5837-xxBA

Commit message: Update Nano-Float_Schematic.kicad_pcb
Parts:
- moved U1 33.9 mm to (114.3, 83.8)
Other:
- board text added: "pressure sensor"
Changed lines of the file:
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@@
   )
   (footprint "Sensor_Pressure:TE_MS5837-xxBA" (layer "F.Cu")
-    (at 147.32 91.44)
+    (at 114.3 83.82)
     (descr "https://www.te.com/commerce/DocumentDelivery/DDEController?Action=showdoc&DocId=Data+Sheet%7FMS5837-30BA%7FB1%7Fpdf%7FEnglish%7FENG_DS_MS5837-30BA_B1.pdf%7FCAT-BLPS0017")
     (tags "MS5837 Ultra-small gel-filled pressure sensor with stainless steel cap")
@@
   (gr_rect (start 76 60.96) (end 101.6 114.3)
     (stroke (width 0.1) (type default)) (fill none) (layer "Edge.Cuts"))
+  (gr_text "pressure sensor\n" (at 111.76 88.9) (layer "Edge.Cuts")
+    (effects (font (size 1 1) (thickness 0.15)) (justify left bottom))
+  )
 )

Commit message: Update Nano-Float_Schematic.kicad_pcb
Parts:
- moved BT1 36.9 mm to (86.5, 99.8), turned to 90 degrees
- moved U1 24.1 mm to (103.1, 62.5)
- moved R1 16.3 mm to (78.7, 99.1)
- moved SW1 12.3 mm to (83.8, 88.9)
- moved DRV8833_H_Bridge1 11.4 mm to (78.7, 86.4)
- moved Fuse1 9.60 mm to (92.6, 91.9)
- moved XIAO_ESP_32C3-RISC-V1 3.59 mm to (86.4, 73.7)
- moved M1 2.54 mm to (78.7, 106.7)
Other:
- board size 25.6 x 53.3 mm -> 20.5 x 48.3 mm
Changed lines of the file:
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@@
   (net 11 "unconnected-(U1-SDA-Pad4)")
   (footprint "Nano-Float_Schematic:SW_ESE-22MV21T" (layer "F.Cu")
-    (at 81.82 101.01)
+    (at 83.82 88.9)
     (property "Sheetfile" "Nano-Float_Schematic.kicad_sch")
     (property "Sheetname" "")
@@
   )
   (footprint "Nano-Float_Schematic:MODULE_102010388" (layer "F.Cu")
-    (at 88.9 76.2)
+    (at 86.36 73.66)
     (property "Sheetfile" "Nano-Float_Schematic.kicad_sch")
     (property "Sheetname" "")
     (attr through_hole)
-    (fp_text reference "XIAO_ESP_32C3-RISC-V1" (at 0 -13.135) (layer "F.SilkS")
+    (fp_text reference "XIAO_ESP_32C3-RISC-V1" (at 0 0 90) (layer "F.SilkS")
         (effects (font (size 1 1) (thickness 0.15)))
     )
@@
   )
   (footprint "Resistor_THT:R_Axial_DIN0207_L6.3mm_D2.5mm_P10.16mm_Horizontal" (layer "F.Cu")
-    (at 88.9 111.76 90)
+    (at 78.74 99.06 90)
     (descr "Resistor, Axial_DIN0207 series, Axial, Horizontal, pin pitch=10.16mm, 0.25W = 1/4W, length*diameter=6.3*2.5mm^2, http://cdn-reichelt.de/documents/datenblatt/B400/1_4W%23YAG.pdf")
     (tags "Resistor Axial_DIN0207 series Axial Horizontal pin pitch 10.16mm 0.25W = 1/4W length 6.3mm diameter 2.5mm")
@@
   )
   (footprint "Connector_PinHeader_2.54mm:PinHeader_2x01_P2.54mm_Vertical" (layer "F.Cu")
-    (at 78.74 109.22)
+    (at 78.74 106.68)
     (descr "Through hole straight pin header, 2x01, 2.54mm pitch, double rows")
     (tags "Through hole pin header THT 2x01 2.54mm double row")
@@
   )
   (footprint "Fuse:Fuseholder_Blade_ATO_Littelfuse_Pudenz_2_Pin" (layer "F.Cu")
-    (at 99.06 99.06 -90)
+    (at 92.64 91.92 -90)
     (descr "Fuseholder ATO Blade littelfuse Pudenz 2 Pin")
     (tags "Fuseholder ATO Blade littelfuse Pudenz 2 Pin")
@@
   )
   (footprint "Battery:Battery_Panasonic_CR1025-VSK_Vertical_CircularHoles" (layer "F.Cu")
-    (at 105.97 68.49)
+    (at 86.47 99.77 90)
     (descr "Panasonic CR-1025/VSK battery")
     (tags "battery CR-1025 coin cell vertical")
@@
     (property "ki_keywords" "batt voltage-source cell")
     (attr through_hole)
-    (fp_text reference "BT1" (at 1.625 -4.3) (layer "F.SilkS")
-        (effects (font (size 1 1) (thickness 0.15)))
-    )
-    (fp_text value "Battery" (at 1.625 1.7) (layer "F.Fab")
-        (effects (font (size 1 1) (thickness 0.15)))
-    )
-    (fp_text user "+" (at -1.46 -0.5) (layer "F.SilkS")
-        (effects (font (size 1 1) (thickness 0.15)))
-    )
-    (fp_text user "${REFERENCE}" (at 1.625 -1.3 180) (layer "F.Fab")
+    (fp_text reference "BT1" (at 1.625 -4.3 90) (layer "F.SilkS")
+        (effects (font (size 1 1) (thickness 0.15)))
+    )
+    (fp_text value "Battery" (at 1.625 1.7 90) (layer "F.Fab")
+        (effects (font (size 1 1) (thickness 0.15)))
+    )
+    (fp_text user "+" (at -1.46 -0.5 90) (layer "F.SilkS")
+        (effects (font (size 1 1) (thickness 0.15)))
+    )
+    (fp_text user "${REFERENCE}" (at 1.625 -1.3 90) (layer "F.Fab")
         (effects (font (size 1 1) (thickness 0.15)))
     )
@@
     (fp_line (start 6.625 -2.75) (end 6.625 0.1)
       (stroke (width 0.1) (type solid)) (layer "F.Fab"))
-    (pad "1" thru_hole rect (at 0 0) (size 1.6 1.6) (drill 1.09) (layers "*.Cu" "*.Mask")
+    (pad "1" thru_hole rect (at 0 0 90) (size 1.6 1.6) (drill 1.09) (layers "*.Cu" "*.Mask")
       (net 1 "VCC") (pinfunction "+") (pintype "passive"))
-    (pad "2" thru_hole circle (at 3.25 -2.65) (size 1.6 1.6) (drill 1.09) (layers "*.Cu" "*.Mask")
+    (pad "2" thru_hole circle (at 3.25 -2.65 90) (size 1.6 1.6) (drill 1.09) (layers "*.Cu" "*.Mask")
       (net 2 "Net-(BT1--)") (pinfunction "-") (pintype "passive"))
     (model "${KICAD6_3DMODEL_DIR}/Battery.3dshapes/Battery_Panasonic_CR1025-VSK_Vertical_CircularHoles.wrl"
@@
   )
   (footprint "Nano-Float_Schematic:SOT5X3-6_DRL_TEX" (layer "F.Cu")
-    (at 88.9 91.44)
+    (at 78.74 86.36)
     (tags "DRV8220DRLR ")
     (property "Sheetfile" "Nano-Float_Schematic.kicad_sch")
@@
         (effects (font (size 1 1) (thickness 0.15)))
     )
-    (fp_text user "${REFERENCE}" (at 0 -2.54 unlocked) (layer "F.Fab")
+    (fp_text user "${REFERENCE}" (at 5.08 -2.54 unlocked) (layer "F.Fab")
         (effects (font (size 1 1) (thickness 0.15)))
     )
@@
   )
   (footprint "Sensor_Pressure:TE_MS5837-xxBA" (layer "F.Cu")
-    (at 114.3 83.82)
+    (at 103.14 62.5)
     (descr "https://www.te.com/commerce/DocumentDelivery/DDEController?Action=showdoc&DocId=Data+Sheet%7FMS5837-30BA%7FB1%7Fpdf%7FEnglish%7FENG_DS_MS5837-30BA_B1.pdf%7FCAT-BLPS0017")
     (tags "MS5837 Ultra-small gel-filled pressure sensor with stainless steel cap")
@@
     )
   )
-  (gr_rect (start 76 60.96) (end 101.6 114.3)
+  (gr_rect (start 76 60.96) (end 96.52 109.22)
     (stroke (width 0.1) (type default)) (fill none) (layer "Edge.Cuts"))
-  (gr_text "pressure sensor\n" (at 111.76 88.9) (layer "Edge.Cuts")
+  (gr_text "pressure sensor\n" (at 100.6 67.58) (layer "Edge.Cuts")
     (effects (font (size 1 1) (thickness 0.15)) (justify left bottom))
   )

Commit message: Update Nano-Float_Schematic.kicad_pcb
Connections:
- U1 pad 1: unconnected-(U1-GND-Pad1) -> GND
- U1 pad 2: unconnected-(U1-VDD-Pad2) -> 3V3
- U1 pad 3: unconnected-(U1-SCL-Pad3) -> Net-(U1-SCL)
- U1 pad 4: unconnected-(U1-SDA-Pad4) -> SDA
Changed lines of the file:
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@@
   (net 6 "3V3")
   (net 7 "D10")
-  (net 8 "unconnected-(U1-GND-Pad1)")
-  (net 9 "unconnected-(U1-VDD-Pad2)")
-  (net 10 "unconnected-(U1-SCL-Pad3)")
-  (net 11 "unconnected-(U1-SDA-Pad4)")
+  (net 8 "Net-(U1-SCL)")
+  (net 9 "SDA")
   (footprint "Nano-Float_Schematic:SW_ESE-22MV21T" (layer "F.Cu")
     (at 83.82 88.9)
@@
         (effects (font (size 1 1) (thickness 0.15)))
     )
-    (fp_text value "~" (at 1.01 11.865) (layer "F.Fab")
+    (fp_text value "~" (at 0 0) (layer "F.Fab")
         (effects (font (size 1 1) (thickness 0.15)))
     )
@@
       (stroke (width 0.1) (type solid)) (fill none) (layer "F.Fab"))
     (pad "1" smd rect (at -1 -1 180) (size 1.3 1.3) (layers "F.Cu" "F.Paste" "F.Mask")
-      (net 8 "unconnected-(U1-GND-Pad1)") (pinfunction "GND") (pintype "power_in"))
+      (net 3 "GND") (pinfunction "GND") (pintype "power_in"))
     (pad "2" smd rect (at -1 1 180) (size 1.3 1.3) (layers "F.Cu" "F.Paste" "F.Mask")
-      (net 9 "unconnected-(U1-VDD-Pad2)") (pinfunction "VDD") (pintype "power_in"))
+      (net 6 "3V3") (pinfunction "VDD") (pintype "power_in"))
     (pad "3" smd rect (at 1 1 180) (size 1.3 1.3) (layers "F.Cu" "F.Paste" "F.Mask")
-      (net 10 "unconnected-(U1-SCL-Pad3)") (pinfunction "SCL") (pintype "passive"))
+      (net 8 "Net-(U1-SCL)") (pinfunction "SCL") (pintype "passive"))
     (pad "4" smd rect (at 1 -1 180) (size 1.3 1.3) (layers "F.Cu" "F.Paste" "F.Mask")
-      (net 11 "unconnected-(U1-SDA-Pad4)") (pinfunction "SDA") (pintype "bidirectional"))
+      (net 9 "SDA") (pinfunction "SDA") (pintype "bidirectional"))
     (model "${KICAD6_3DMODEL_DIR}/Sensor_Pressure.3dshapes/TE_MS5837-xxBA.wrl"
       (offset (xyz 0 0 0))

Commit message: footprints? yes!
Parts:
- added C1: C_Small, Capacitor_THT:C_Disc_D3.0mm_W1.6mm_P2.50mm, F.Cu at (94.0, 88.9)
- added R2: R, Resistor_THT:R_Axial_DIN0207_L6.3mm_D2.5mm_P10.16mm_Horizontal, F.Cu at (83.8, 94.0)
- added R3: R, Resistor_THT:R_Axial_DIN0207_L6.3mm_D2.5mm_P10.16mm_Horizontal, F.Cu at (83.8, 99.1)
- Fuse1: footprint Fuse:Fuseholder_Blade_ATO_Littelfuse_Pudenz_2_Pin -> TestPoint:TestPoint_2Pads_Pitch2.54mm_Drill0.8mm
- moved U1 30.8 mm to (110.2, 92.4)
- moved BT1 7.32 mm to (88.9, 106.7), turned to 0 degrees
- moved Fuse1 6.70 mm to (88.9, 86.4)
- moved M1 2.54 mm to (78.7, 104.1)
- moved SW1 0.59 mm to (83.8, 88.3)
