File: FloatSID.kicad_sch (KiCad schematic)
At the start: 14 parts, among them M1 Motor_DC, SW1 SW, SW2 Limit Switch, U1 Custom PCB, U2 XiaoESP32C3, U3 MS583730BA01-50

Commit message: my float pcb work
Parts:
- B1: footprint (none) -> Battery:Battery_Panasonic_CR1025-VSK_Vertical_CircularHoles
- C1: footprint (none) -> Capacitor_THT:C_Disc_D3.0mm_W1.6mm_P2.50mm
- HBridge1: footprint (none) -> Nano-Float_Schematic FR:SOT5X3-6_DRL_TEX
- U2: footprint (none) -> Nano-Float_Schematic FR:MODULE_102010388
Connections:
- new net: D1.1 (K), HBridge1. (VDD), U1. (OUT-)
Changed lines of the file:
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@@
       (effects (font (size 1.27 1.27)))
     )
-    (property "Footprint" "" (at 165.1 113.03 0)
+    (property "Footprint" "Nano-Float_Schematic FR:SOT5X3-6_DRL_TEX" (at 165.1 113.03 0)
       (effects (font (size 1.27 1.27)) hide)
     )
@@
       (effects (font (size 1.27 1.27)) (justify left) hide)
     )
-    (property "Footprint" "" (at 47.625 88.265 0)
+    (property "Footprint" "Capacitor_THT:C_Disc_D3.0mm_W1.6mm_P2.50mm" (at 47.625 88.265 0)
       (effects (font (size 1.27 1.27)) hide)
     )
@@
       (effects (font (size 2 2)))
     )
-    (property "Footprint" "" (at 130.175 98.425 0)
+    (property "Footprint" "Nano-Float_Schematic FR:MODULE_102010388" (at 130.175 98.425 0)
       (effects (font (size 1.27 1.27)) (justify bottom) hide)
     )
@@
       (effects (font (size 2 2)) (justify left))
     )
-    (property "Footprint" "" (at 27.94 90.551 90)
+    (property "Footprint" "Battery:Battery_Panasonic_CR1025-VSK_Vertical_CircularHoles" (at 27.94 90.551 90)
       (effects (font (size 1.27 1.27)) hide)
     )
