File: FloatSIDBasedPCBAlt/FloatSID.kicad_pcb (KiCad board)
At the start: 2 copper layers, 6 parts, among them U2 XiaoESP32C3

Commit message: Float PCB Updates
Parts:
- removed B1: 1.5V, Battery:Battery_Panasonic_CR1025-VSK_Vertical_CircularHoles
- added B4: 1.5V, Connector_PinHeader_2.54mm:PinHeader_1x02_P2.54mm_Vertical, F.Cu at (100.8, 101.7)
- added C2: C_Small, Capacitor_SMD:C_1812_4532Metric_Pad1.57x3.40mm_HandSolder, F.Cu at (125.7, 92.3)
- added C3: C_Small, Capacitor_SMD:C_1812_4532Metric_Pad1.57x3.40mm_HandSolder, F.Cu at (121.7, 92.3)
- added C4: C_Small, Capacitor_SMD:C_1812_4532Metric_Pad1.57x3.40mm_HandSolder, F.Cu at (123.0, 87.1)
- added F1: 2A Fuse, MINI-Fuse-Holder-H:FUSE_01530007Z, F.Cu at (125.7, 105.3)
- added M1: Motor_DC, Connector_PinHeader_2.54mm:PinHeader_1x02_P2.54mm_Vertical, F.Cu at (148.1, 75.2)
- added R1: 220kOhm, Resistor_THT:R_Axial_DIN0207_L6.3mm_D2.5mm_P7.62mm_Horizontal, F.Cu at (136.6, 74.9)
- added R2: 220kOhm, Resistor_THT:R_Axial_DIN0207_L6.3mm_D2.5mm_P7.62mm_Horizontal, F.Cu at (136.6, 79.0)
- added R3: 10kOhm, Resistor_THT:R_Axial_DIN0207_L6.3mm_D2.5mm_P7.62mm_Horizontal, F.Cu at (105.6, 87.6)
- added R4: 10kOhm, Resistor_THT:R_Axial_DIN0207_L6.3mm_D2.5mm_P7.62mm_Horizontal, F.Cu at (136.6, 87.0)
- added SW1: SW, Button_Switch_THT:SW_09.10290.01_EAO, F.Cu at (125.6, 119.7)
- added SW2: Limit Switch, Connector_PinHeader_2.54mm:PinHeader_1x02_P2.54mm_Vertical, F.Cu at (152.7, 75.2)
- added U4: XiaoESP32C3, XIAO_ESP32C3:XIAO_ESP32C3_THT, F.Cu at (125.6, 87.9)
- C1: footprint Capacitor_THT:C_Disc_D3.0mm_W1.6mm_P2.50mm -> Capacitor_SMD:C_1812_4532Metric_Pad1.57x3.40mm_HandSolder
- HBridge1: footprint Nano-Float_Schematic FR:SOT5X3-6_DRL_TEX -> NanoFloat Pressure Sensor:DRV8220DRLR
- U2: value XiaoESP32C3 -> MS583730BA01-50; footprint Nano-Float_Schematic FR:MODULE_102010388 -> Connector_PinHeader_1.00mm:PinHeader_2x02_P1.00mm_Vertical
- moved D2 117.1 mm to (142.7, 116.9), turned to 90 degrees
- moved U2 107.0 mm to (147.4, 85.5)
- moved D1 101.8 mm to (136.9, 91.2)
- moved C1 94.1 mm to (129.7, 92.3), turned to 90 degrees
- moved HBridge1 86.8 mm to (129.8, 85.7)
Connections:
- C1 pad 2: Net-(U1-GND) -> Net-(D1-K)
- U2 pad 2: unconnected-(U2-D1-Pad2) -> Net-(U2-VDD)
- U2 pad 3: unconnected-(U2-D2-Pad3) -> Net-(U2-SCL)
- U2 pad 4: unconnected-(U2-D3-Pad4) -> Net-(U2-SDA)
