File: FloatSIDBasedPCBAlt/FloatSID.kicad_sch (KiCad schematic)
At the start: 14 parts, among them M1 Motor_DC, SW1 SW, SW2 Limit Switch, U1 Custom PCB, U2 XiaoESP32C3, U3 MS583730BA01-50

Commit message: Float PCB Updates
Parts:
- removed U1: Custom PCB, 113991054:MODULE_113991054, symbol 113991054:113991054
- added C2, C3, C4: C_Small, Capacitor_SMD:C_1812_4532Metric_Pad1.57x3.40mm_HandSolder, symbol Device:C_Small
- added R3, R4: 10kOhm, Resistor_THT:R_Axial_DIN0207_L6.3mm_D2.5mm_P7.62mm_Horizontal, symbol Device:R_Small
- B4: renamed from B1; footprint Battery:Battery_Panasonic_CR1025-VSK_Vertical_CircularHoles -> Connector_PinHeader_2.54mm:PinHeader_1x02_P2.54mm_Vertical
- C1: footprint Capacitor_THT:C_Disc_D3.0mm_W1.6mm_P2.50mm -> Capacitor_SMD:C_1812_4532Metric_Pad1.57x3.40mm_HandSolder
- F1: footprint (none) -> MINI-Fuse-Holder-H:FUSE_01530007Z
- HBridge1: footprint Nano-Float_Schematic FR:SOT5X3-6_DRL_TEX -> NanoFloat Pressure Sensor:DRV8220DRLR
- M1, SW2: footprint (none) -> Connector_PinHeader_2.54mm:PinHeader_1x02_P2.54mm_Vertical
- R1, R2: footprint (none) -> Resistor_THT:R_Axial_DIN0207_L6.3mm_D2.5mm_P7.62mm_Horizontal
- SW1: footprint (none) -> Button_Switch_THT:SW_09.10290.01_EAO
- U2: renamed from U3; footprint (none) -> Connector_PinHeader_1.00mm:PinHeader_2x02_P1.00mm_Vertical
- U4: renamed from U2; footprint Nano-Float_Schematic FR:MODULE_102010388 -> XIAO_ESP32C3:XIAO_ESP32C3_THT
Connections:
- net at U2.1 (GND), U4.13 (GND): now also C4.2
- net at U2.2 (VDD), U4.12 (VCC_3V3): now also C4.1, R3.1, R4.2
- net at U2.3 (SCL), U4.6 (D5_SCL): now also R4.1
- net at U2.4 (SDA), U4.5 (D4_SDA): now also R3.2
- net at D1.1 (K), HBridge1. (VDD): now also C1.2, F1.1, C2.2, C3.1
- net at SW1.2 (B): now also HBridge1. (VDD), R1.1, U4. (BAT-), C2.1, C3.2
Other:
- moved on the sheet: B4
