File: NanoBoard/NB002/NB002.kicad_pcb (KiCad board)
At the start: 2 copper layers, 22 x 72.8 mm, 18 parts, among them M1 Motor_DC, SW1 SW, SW2 Limit Switch, U2 MS583730BA01-50, U4 XiaoESP32C3

Commit message: Updated Ground Planes
Connections:
- C4 pad 2: Net-(B4--) -> Net-(D1-K)
- U2 pad 1: Net-(B4--) -> Net-(D1-K)
- U4 pad GND: Net-(B4--) -> Net-(D1-K)
Routing:
- net Net-(D1-K): track 73.5 -> 0.00 mm, vias 1 -> 42
- net Net-(B4--): track 0.00 -> 60.1 mm, vias 64 -> 0
- net Net-(U2-VDD): track 121.5 -> 122.1 mm
- added copper zone on B.Cu, net Net-(D1-K)
- added copper zone on F.Cu, net Net-(D1-K)
- removed copper zone on B.Cu, net Net-(B4--)
- removed copper zone on F.Cu, net Net-(B4--)
Other:
- outline, holes or cut-outs redrawn
