File: NanoBoard/NB102/NB102.kicad_pcb (KiCad board)
At the start: 2 copper layers, 22 x 70.3 mm, 18 parts, among them M1 Motor_DC, SW1 SW, SW2 Limit Switch, U1 XiaoESP32C6, U2 MS583730BA01-50, U3 DRV8833-THT

Commit message: Updates to boards and Flashing Micropython
Parts:
- removed C1, C2, C3: C_Small, Capacitor_SMD:C_1812_4532Metric_Pad1.57x3.40mm_HandSolder
- added LED: PinHeader_1x02_P2.00mm_Vertical, Connector_PinHeader_2.00mm:PinHeader_1x02_P2.00mm_Vertical, B.Cu at (145.3, 75.2)
- added M1: PinHeader_2x03_P2.00mm_Vertical, Connector_PinHeader_2.00mm:PinHeader_2x03_P2.00mm_Vertical, F.Cu at (145.5, 117.4)
- moved F1 4.30 mm to (140.1, 110.7)
- moved REF** 0.50 mm to (149.1, 68.7)
- renumbered M1 to J1
Connections:
- BAT pad 1: Net-(B1-+) -> Net-(SW1-B)
- J1 pad 1: Net-(M1-+) -> (no net)
- J1 pad 2: Net-(M1--) -> (no net)
Routing:
- net unconnected-(U1-D2-Pad3): track 0.00 -> 65.6 mm, vias 0 -> 2
- net unconnected-(U1-D1-Pad2): track 0.00 -> 61.6 mm, vias 0 -> 2
- net Net-(D1-K): track 69.1 -> 13.9 mm, vias 70 -> 67
- net Net-(B1-+): track 64.6 -> 16.6 mm, vias 1 -> 0
- net Net-(SW1-B): track 72.9 -> 48.4 mm, vias 1 -> 2
- net Net-(M1-+): track 29.1 -> 19.2 mm
- net Net-(U1-GND): track 57.2 -> 66.4 mm
- net Net-(U1-VCC_3V3): track 49.8 -> 58.0 mm
- net Net-(U1-D9): track 29.3 -> 22.5 mm
- net Net-(M1--): track 26.1 -> 20.5 mm
- net Net-(B1--): track 17.1 -> 22.4 mm
- net Net-(SW2-COM): track 52.9 -> 53.6 mm
- net Net-(D1-A): track 13.3 -> 12.8 mm
Other:
- outline, holes or cut-outs redrawn
- board text added: "+"
- board text added: "-"
